Commit message: unification of sim and bags, update of docs

File: src/minidog_sim/urdf/diffbot.urdf.xacro (robot description, xacro)
@@ -35,6 +35,5 @@
     </inertial>
   </xacro:macro>
-  <!-- Frames -->
-  <link name="base_footprint"/>
+  <!-- Root frame: base_link (matches real GO2 convention, no base_footprint) -->
   <link name="base_link">
     <visual>
@@ -55,9 +54,4 @@
     <xacro:inertial_box mass="5.0" x="${chassis_length}" y="${chassis_width}" z="${chassis_height}"/>
   </link>
-  <joint name="base_footprint_joint" type="fixed">
-    <parent link="base_footprint"/>
-    <child link="base_link"/>
-    <origin xyz="0 0 ${base_z}" rpy="0 0 0"/>
-  </joint>
   <!-- Left drive wheel -->
   <link name="left_wheel_link">
@@ -195,5 +189,5 @@
       <dimensions>3</dimensions>
       <odom_frame>odom</odom_frame>
-      <robot_base_frame>base_footprint</robot_base_frame>
+      <robot_base_frame>base_link</robot_base_frame>
       <odom_publish_frequency>50</odom_publish_frequency>
     </plugin>
